File: scheme/Awtr/Awtr.kicad_sch (KiCad schematic)
At the start: 12 parts, among them J1 Barrel_Jack_Switch, J2 WCH_Link, J3 Water_pump, J4 Sensor, Q1 IRLB8743, SW1 SW_Push, U1 CH32V003J4M6

Commit message: +ADC
Parts:
- added C1: 10pF, Capacitor_THT:C_Disc_D5.0mm_W2.5mm_P5.00mm, symbol Device:C
Connections:
- net GND: now also C1.2
- net at SW1.2, U1.7 (PC4): now also C1.1
Other:
- moved on the sheet: SW1
Changed lines of the file:
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@@
 	(paper "A4")
+	(junction
+		(at 104.14 82.55)
+		(diameter 0)
+		(color 0 0 0 0)
+	)
+	(junction
+		(at 104.14 95.25)
+		(diameter 0)
+		(color 0 0 0 0)
+	)
 	(junction
 		(at 220.98 74.93)
@@
 	(wire
 		(pts
-			(xy 101.6 95.25) (xy 124.46 95.25)
+			(xy 90.17 95.25) (xy 104.14 95.25)
 		)
 		(stroke
@@
 	(wire
 		(pts
+			(xy 104.14 82.55) (xy 90.17 82.55)
+		)
+		(stroke
+			(width 0)
+			(type default)
+		)
+	)
+	(wire
+		(pts
 			(xy 78.74 78.74) (xy 80.01 78.74)
 		)
@@
 	(wire
 		(pts
-			(xy 101.6 93.98) (xy 101.6 95.25)
+			(xy 90.17 93.98) (xy 90.17 95.25)
 		)
 		(stroke
@@
 	(wire
 		(pts
-			(xy 101.6 82.55) (xy 101.6 83.82)
+			(xy 104.14 95.25) (xy 124.46 95.25)
+		)
+		(stroke
+			(width 0)
+			(type default)
+		)
+	)
+	(wire
+		(pts
+			(xy 104.14 82.55) (xy 104.14 85.09)
+		)
+		(stroke
+			(width 0)
+			(type default)
+		)
+	)
+	(wire
+		(pts
+			(xy 90.17 82.55) (xy 90.17 83.82)
 		)
 		(stroke
@@
 	(wire
 		(pts
+			(xy 104.14 92.71) (xy 104.14 95.25)
+		)
+		(stroke
+			(width 0)
+			(type default)
+		)
+	)
+	(wire
+		(pts
 			(xy 156.21 81.28) (xy 158.75 81.28)
 		)
@@
 	(wire
 		(pts
-			(xy 106.68 82.55) (xy 101.6 82.55)
+			(xy 106.68 82.55) (xy 104.14 82.55)
 		)
 		(stroke
@@
 				(path "/a526cc2a-2896-44f6-895f-0822ab62eb25"
 					(reference "#PWR04")
+					(unit 1)
+				)
+			)
+		)
+	)
+	(symbol
+		(lib_id "Device:C")
+		(at 104.14 88.9 0)
+		(unit 1)
+		(exclude_from_sim no)
+		(in_bom yes)
+		(on_board yes)
+		(dnp no)
+		(fields_autoplaced yes)
+		(property "Reference" "C1"
+			(at 107.95 87.6299 0)
+			(effects
+				(font
+					(size 1.27 1.27)
+				)
+				(justify left)
+			)
+		)
+		(property "Value" "10pF"
+			(at 107.95 90.1699 0)
+			(effects
+				(font
+					(size 1.27 1.27)
+				)
+				(justify left)
+			)
+		)
+		(property "Footprint" "Capacitor_THT:C_Disc_D5.0mm_W2.5mm_P5.00mm"
+			(at 105.1052 92.71 0)
+			(effects
+				(font
+					(size 1.27 1.27)
+				)
+				(hide yes)
+			)
+		)
+		(property "Datasheet" "~"
+			(at 104.14 88.9 0)
+			(effects
+				(font
+					(size 1.27 1.27)
+				)
+				(hide yes)
+			)
+		)
+		(property "Description" "Unpolarized capacitor"
+			(at 104.14 88.9 0)
+			(effects
+				(font
+					(size 1.27 1.27)
+				)
+				(hide yes)
+			)
+		)
+		(pin "1"
+		)
+		(pin "2"
+		)
+		(instances
+			(project ""
+				(path "/a526cc2a-2896-44f6-895f-0822ab62eb25"
+					(reference "C1")
 					(unit 1)
 				)
@@
 	(symbol
 		(lib_id "Switch:SW_Push")
-		(at 101.6 88.9 90)
+		(at 90.17 88.9 90)
 		(unit 1)
 		(exclude_from_sim no)
@@
 		(fields_autoplaced yes)
 		(property "Reference" "SW1"
-			(at 102.87 87.6299 90)
+			(at 91.44 87.6299 90)
 			(effects
 				(font
@@
 		)
 		(property "Value" "SW_Push"
-			(at 102.87 90.1699 90)
+			(at 91.44 90.1699 90)
 			(effects
 				(font
@@
 		)
 		(property "Footprint" "Button_Switch_SMD:SW_Push_1TS009xxxx-xxxx-xxxx_6x6x5mm"
-			(at 96.52 88.9 0)
+			(at 85.09 88.9 0)
 			(effects
 				(font
@@
 		)
 		(property "Datasheet" "~"
-			(at 96.52 88.9 0)
+			(at 85.09 88.9 0)
 			(effects
 				(font
@@
 		)
 		(property "Description" "Push button switch, generic, two pins"
-			(at 101.6 88.9 0)
-			(effects
-				(font
+			(at 90.17 88.9 0)
+			(effects
+				(font
